File: M4_CAN_Feather_Carrier.kicad_pcb (KiCad board)
At the start: 4 copper layers, 70.5 x 79.5 mm, 68 parts, among them J1 2601-3102, J2 2601-3103, J3 conn_04_03, J4 Conn_02x04_Odd_Even, J5 Conn_01x03, J6 Conn_01x02, J7 conn_04_03, U1 LMR33630BDDA, U2 Feather_M4_CAN_Express, U3 TXS0104EPW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

Commit message: KiCAD files (initial)
Parts:
- added C11: 0.1u, Capacitor_SMD:C_0603_1608Metric, F.Cu at (63.4, 7.90)
- added IC1: 74LVC2G17GV,125, Appreciate:SOT95P275X110-6N, F.Cu at (65.3, 11.4)
- C1, C26: footprint Appreciate:CAPAE830X1050N -> Capacitor_SMD:CP_Elec_8x10
- moved REF** 2.72 mm to (64.2, 4.00)
- moved C25 1.41 mm to (65.6, 17.5)
Connections:
- J2 pad 1: /NEOPIXEL -> Net-(IC1-1Y)
- J2 pad 2: /NEOPIXEL -> Net-(IC1-1Y)
Routing:
- net Net-(IC1-1Y): track 0.00 -> 19.9 mm
- net GND: track 90.0 -> 95.8 mm, vias 38 -> 40
- net +5V: track 5.75 -> 10.5 mm, vias 16 -> 17
- net /NEOPIXEL: track 65.9 -> 64.9 mm
