File: M4_CAN_Feather_Carrier.kicad_sch (KiCad schematic)
At the start: 67 parts, among them J1 2601-3102, J2 2601-3103, J3 conn_04_03, J4 Conn_02x04_Odd_Even, J5 Conn_01x03, J6 Conn_01x02, J7 conn_04_03, U1 LMR33630BDDA, U2 Feather_M4_CAN_Express, U3 TXS0104EPW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

Commit message: KiCAD files (initial)
Parts:
- added C11: 0.1u, Capacitor_SMD:C_0603_1608Metric, symbol Device:C_Small
- added IC1: 74LVC2G17GV,125, Appreciate:SOT95P275X110-6N, symbol Appreciate:74LVC2G17GV,125
- C1, C26: footprint Appreciate:CAPAE830X1050N -> Capacitor_SMD:CP_Elec_8x10; LCSC C340767 -> C2164760
Connections:
- net +5V: now also C11.1, IC1.5 (VCC)
- net GND: now also C11.2, IC1.2 (GND), IC1.3 (2A)
- net NEOPIXEL: now also IC1.1 (1A); no longer J2.1 (1.1), J2.2 (1.2)
- new net: IC1.6 (1Y), J2.1 (1.1), J2.2 (1.2)
- no-connect marks 33 -> 34
Other:
- moved on the sheet: C1, C2, C3, C6, C7, C8, C9, D101, J2, L1, U1, X2
